File: docs/schematics/sound trigger sensor/sound trigger sensor.kicad_sch (KiCad schematic)
At the start: 14 parts, among them J1 Conn_01x03_Pin, Q1 NPN, U1 LM393

Commit message: nicer schematic explanations
Connections:
- net VREF: now reaches RV1.2, U1.2 (-)
Other:
- note added: "Bias voltage for the electret mic"
- note added: "Common-emitter amplifier + low-pass (R1+C2)"
- note added: "DC block"
- note added: "OUT level: 0V = sound detected VCC = no sound detected"
- note added: "Sound Sensor Module"
- note added: "Threshold voltage"
- note added: "by: spezifisch+ee@gmail.com License: CERN-OHL-S-2.0"
- note added: "v1.0"
Changed lines of the file:
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@@
 	(wire
 		(pts
-			(xy 158.75 125.73) (xy 158.75 123.19)
+			(xy 158.75 128.27) (xy 158.75 123.19)
 		)
 		(stroke
@@
 	(wire
 		(pts
-			(xy 167.64 119.38) (xy 162.56 119.38)
-		)
-		(stroke
-			(width 0)
-			(type default)
-		)
-	)
-	(wire
-		(pts
-			(xy 167.64 109.22) (xy 170.18 109.22)
-		)
-		(stroke
-			(width 0)
-			(type default)
-		)
-	)
-	(wire
-		(pts
-			(xy 140.97 119.38) (xy 140.97 125.73)
+			(xy 163.83 119.38) (xy 162.56 119.38)
+		)
+		(stroke
+			(width 0)
+			(type default)
+		)
+	)
+	(wire
+		(pts
+			(xy 163.83 109.22) (xy 170.18 109.22)
+		)
+		(stroke
+			(width 0)
+			(type default)
+		)
+	)
+	(wire
+		(pts
+			(xy 140.97 119.38) (xy 140.97 128.27)
 		)
 		(stroke
@@
 	(wire
 		(pts
-			(xy 167.64 119.38) (xy 167.64 109.22)
+			(xy 163.83 109.22) (xy 163.83 119.38)
 		)
 		(stroke
@@
 			(width 0)
 			(type default)
+		)
+	)
+	(rectangle
+		(start 81.915 82.55)
+		(end 103.505 123.825)
+		(stroke
+			(width 0)
+			(type dash)
+			(color 72 72 72 1)
+		)
+		(fill
+			(type none)
+		)
+	)
+	(rectangle
+		(start 117.475 82.55)
+		(end 147.955 123.825)
+		(stroke
+			(width 0)
+			(type dash)
+			(color 72 72 72 1)
+		)
+		(fill
+			(type none)
+		)
+	)
+	(rectangle
+		(start 111.125 101.6)
+		(end 111.125 101.6)
+		(stroke
+			(width 0)
+			(type default)
+		)
+		(fill
+			(type none)
+		)
+	)
+	(rectangle
+		(start 107.95 101.6)
+		(end 116.84 115.57)
+		(stroke
+			(width 0)
+			(type dash)
+			(color 72 72 72 1)
+		)
+		(fill
+			(type none)
+		)
+	)
+	(text "by: spezifisch+ee@gmail.com\nLicense: CERN-OHL-S-2.0"
+		(exclude_from_sim no)
+		(at 255.778 179.324 0)
+		(effects
+			(font
+				(size 1.27 1.27)
+				(color 132 0 0 1)
+			)
+			(justify left)
+		)
+	)
+	(text "Threshold voltage"
+		(exclude_from_sim no)
+		(at 162.306 121.92 0)
+		(effects
+			(font
+				(size 1.27 1.27)
+				(color 72 72 72 1)
+			)
+			(justify left)
+		)
+	)
+	(text "Sound Sensor Module"
+		(exclude_from_sim no)
+		(at 187.452 189.738 0)
+		(effects
+			(font
+				(size 1.905 1.905)
+				(color 132 0 0 1)
+			)
+			(justify left)
+		)
+	)
+	(text "v1.0"
+		(exclude_from_sim no)
+		(at 268.478 193.294 0)
+		(effects
+			(font
+				(size 1.27 1.27)
+				(color 132 0 0 1)
+			)
+			(justify left)
+		)
+	)
+	(text "OUT level:\n0V = sound detected\nVCC = no sound detected"
+		(exclude_from_sim no)
+		(at 198.12 116.84 0)
+		(effects
+			(font
+				(size 1.27 1.27)
+				(color 72 72 72 1)
+			)
+			(justify left)
+		)
+	)
+	(text "Bias voltage for the electret mic"
+		(exclude_from_sim no)
+		(at 81.534 125.73 0)
+		(effects
+			(font
+				(size 1.27 1.27)
+				(color 72 72 72 1)
+			)
+			(justify left)
+		)
+	)
+	(text "Common-emitter amplifier\n+ low-pass (R1+C2)"
+		(exclude_from_sim no)
+		(at 117.602 126.746 0)
+		(effects
+			(font
+				(size 1.27 1.27)
+				(color 72 72 72 1)
+			)
+			(justify left)
+		)
+	)
+	(text "DC block"
+		(exclude_from_sim no)
+		(at 107.95 117.348 0)
+		(effects
+			(font
+				(size 1.27 1.27)
+				(color 72 72 72 1)
+			)
+			(justify left)
 		)
 	)
 	(label "OUT"
 		(at 198.12 106.68 0)
+		(fields_autoplaced yes)
+		(effects
+			(font
+				(size 1.27 1.27)
+			)
+			(justify left bottom)
+		)
+	)
+	(label "VREF"
+		(at 163.83 109.22 0)
 		(fields_autoplaced yes)
 		(effects
@@
 	(symbol
 		(lib_id "power:GND")
-		(at 140.97 125.73 0)
+		(at 140.97 128.27 0)
 		(unit 1)
 		(exclude_from_sim no)
@@
 		(fields_autoplaced yes)
 		(property "Reference" "#PWR07"
-			(at 140.97 132.08 0)
+			(at 140.97 134.62 0)
 			(effects
 				(font
@@
 		)
 		(property "Value" "GND"
-			(at 140.97 130.81 0)
+			(at 140.97 133.35 0)
 			(effects
 				(font
@@
 		)
 		(property "Footprint" ""
-			(at 140.97 125.73 0)
+			(at 140.97 128.27 0)
 			(effects
 				(font
@@
 		)
 		(property "Datasheet" ""
-			(at 140.97 125.73 0)
+			(at 140.97 128.27 0)
 			(effects
 				(font
@@
 		)
 		(property "Description" "Power symbol creates a global label with name \"GND\" , ground"
-			(at 140.97 125.73 0)
+			(at 140.97 128.27 0)
 			(effects
 				(font
@@
 	(symbol
 		(lib_id "power:GND")
-		(at 158.75 125.73 0)
+		(at 158.75 128.27 0)
 		(unit 1)
 		(exclude_from_sim no)
@@
 		(fields_autoplaced yes)
 		(property "Reference" "#PWR01"
-			(at 158.75 132.08 0)
+			(at 158.75 134.62 0)
 			(effects
 				(font
@@
 		)
 		(property "Value" "GND"
-			(at 158.75 130.81 0)
+			(at 158.75 133.35 0)
 			(effects
 				(font
@@
 		)
 		(property "Footprint" ""
-			(at 158.75 125.73 0)
+			(at 158.75 128.27 0)
 			(effects
 				(font
@@
 		)
 		(property "Datasheet" ""
-			(at 158.75 125.73 0)
+			(at 158.75 128.27 0)
 			(effects
 				(font
@@
 		)
 		(property "Description" "Power symbol creates a global label with name \"GND\" , ground"
-			(at 158.75 125.73 0)
-			(effects
-				(font
+			(at 158.75 128.27 0)
+			(effects
+				(font
